File: Gardening-pHAT.kicad_pcb (KiCad board)
At the start: 2 copper layers, 65 x 30 mm, 25 parts, among them P1 CONN_01X03, P2 CONN_01X03, P3 CONN_01X03, P4 CONN_02X05, U1 CAT24C32WI-GT3, U2 MCP3002

Commit message: Update routing again
Signed-off-by: Leon Anavi <leon@anavi.org>
Parts:
- moved C1 1.14 mm to (211.8, 84.7)
- moved R3 1.08 mm to (208.8, 84.8)
- moved R1 1.02 mm to (211.8, 89.9)
- moved R2 0.95 mm to (208.8, 89.9)
Connections:
- RASP_CONN1 pad 11: Net-(P4-Pad3) -> Net-(P4-Pad5)
- RASP_CONN1 pad 13: Net-(P4-Pad5) -> Net-(P4-Pad3)
- RASP_CONN1 pad 17: (no net) -> +3V3
Routing:
- net +3V3: track 151.8 -> 162.7 mm
- net Net-(P4-Pad3): track 26.2 -> 36.7 mm, vias 1 -> 0
- net GND: track 0.00 -> 5.64 mm
- net Net-(JP1-Pad1): track 31.9 -> 29.0 mm
- net Net-(P4-Pad5): track 28.0 -> 30.3 mm, vias 2 -> 0
- net Net-(R4-Pad2): track 38.6 -> 41.0 mm
- net Net-(R3-Pad2): track 33.1 -> 35.5 mm, vias 1 -> 2
- net Net-(R5-Pad2): track 18.0 -> 16.8 mm
- net Net-(P4-Pad1): track 46.2 -> 47.1 mm
Other:
- board text added: "G18 G27 G17 5V 5V"
- board text removed: "G18 G17 G27 5V 5V"

Commit message: Add junction between 5V pins on the header
Signed-off-by: Leon Anavi <leon@anavi.org>
Connections:
- RASP_CONN1 pad 4: (no net) -> +5V
Changed lines of the file:
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@@
 (kicad_pcb (version 4) (host pcbnew 4.0.4+dfsg1-stable)
   (general
-    (links 70)
-    (no_connects 1)
-    (area 148.451099 74.953599 213.551101 105.053601)
+    (links 71)
+    (no_connects 2)
+    (area 136.817429 66.3 225.182572 106.680001)
     (thickness 1.6)
     (drawings 32)
@@
     (pad 3 thru_hole oval (at 0 2.54 90) (size 1.7272 1.7272) (drill 1.016) (layers *.Cu *.Mask F.SilkS)
       (net 7 "Net-(R6-Pad2)"))
-    (pad 4 thru_hole oval (at 2.54 2.54 90) (size 1.7272 1.7272) (drill 1.016) (layers *.Cu *.Mask F.SilkS))
+    (pad 4 thru_hole oval (at 2.54 2.54 90) (size 1.7272 1.7272) (drill 1.016) (layers *.Cu *.Mask F.SilkS)
+      (net 3 +5V))
     (pad 5 thru_hole oval (at 0 5.08 90) (size 1.7272 1.7272) (drill 1.016) (layers *.Cu *.Mask F.SilkS)
       (net 8 "Net-(R7-Pad2)"))
