File: Gardening-pHAT.sch (KiCad schematic (older format))
At the start: 20 parts, among them P1 CONN_01X03, P2 CONN_01X03, P3 CONN_01X03, P4 CONN_02X05, U1 CAT24C32WI-GT3, U2 MCP3002

Commit message: Fix routing
Signed-off-by: Leon Anavi <leon@anavi.org>
Connections:
- net +3V3: no longer RASP_CONN1.17 (VDD(3.3V))
- net +5V: no longer RASP_CONN1.4 (Vpp(5V))
- no-connect marks 13 -> 15
Changed lines of the file:
@@
 $EndComp
 $Comp
-L GND #PWR1
+L GND #PWR01
 U 1 1 56FB5AA8
 P 800 3950
-F 0 "#PWR1" H 800 3700 50  0001 C CNN
+F 0 "#PWR01" H 800 3700 50  0001 C CNN
 F 1 "GND" H 800 3800 50  0000 C CNN
 F 2 "" H 800 3950 50  0000 C CNN
@@
 $EndComp
 $Comp
-L GND #PWR2
+L GND #PWR02
 U 1 1 56FB5B93
 P 1900 3050
-F 0 "#PWR2" H 1900 2800 50  0001 C CNN
+F 0 "#PWR02" H 1900 2800 50  0001 C CNN
 F 1 "GND" H 1900 2900 50  0000 C CNN
 F 2 "" H 1900 3050 50  0000 C CNN
@@
 $EndComp
 $Comp
-L +3.3V #PWR3
+L +3.3V #PWR03
 U 1 1 56FB5F37
 P 2200 2700
-F 0 "#PWR3" H 2200 2550 50  0001 C CNN
+F 0 "#PWR03" H 2200 2550 50  0001 C CNN
 F 1 "+3.3V" H 2200 2840 50  0000 C CNN
 F 2 "" H 2200 2700 50  0000 C CNN
@@
 $EndComp
 $Comp
-L GND #PWR4
+L GND #PWR04
 U 1 1 56FB60BD
 P 2650 4650
-F 0 "#PWR4" H 2650 4400 50  0001 C CNN
+F 0 "#PWR04" H 2650 4400 50  0001 C CNN
 F 1 "GND" H 2650 4500 50  0000 C CNN
 F 2 "" H 2650 4650 50  0000 C CNN
@@
 $EndComp
 $Comp
-L GND #PWR7
+L GND #PWR05
 U 1 1 56FD1B71
 P 3450 3450
-F 0 "#PWR7" H 3450 3200 50  0001 C CNN
+F 0 "#PWR05" H 3450 3200 50  0001 C CNN
 F 1 "GND" H 3450 3300 50  0000 C CNN
 F 2 "" H 3450 3450 50  0000 C CNN
@@
 $EndComp
 $Comp
-L +3.3V #PWR6
+L +3.3V #PWR06
 U 1 1 56FD2267
 P 3450 2150
-F 0 "#PWR6" H 3450 2000 50  0001 C CNN
+F 0 "#PWR06" H 3450 2000 50  0001 C CNN
 F 1 "+3.3V" H 3450 2290 50  0000 C CNN
 F 2 "" H 3450 2150 50  0000 C CNN
@@
 $EndComp
 $Comp
-L +5V #PWR5
+L +5V #PWR07
 U 1 1 56FF1D94
 P 3450 1800
-F 0 "#PWR5" H 3450 1650 50  0001 C CNN
+F 0 "#PWR07" H 3450 1650 50  0001 C CNN
 F 1 "+5V" H 3450 1940 50  0000 C CNN
 F 2 "" H 3450 1800 50  0000 C CNN
@@
 $EndComp
 $Comp
-L GND #PWR19
+L GND #PWR08
 U 1 1 5704B80C
 P 8050 2100
-F 0 "#PWR19" H 8050 1850 50  0001 C CNN
+F 0 "#PWR08" H 8050 1850 50  0001 C CNN
 F 1 "GND" H 8050 1950 50  0000 C CNN
 F 2 "" H 8050 2100 50  0000 C CNN
@@
 $EndComp
 $Comp
-L +3.3V #PWR18
+L +3.3V #PWR09
 U 1 1 5704BA43
 P 7900 1200
-F 0 "#PWR18" H 7900 1050 50  0001 C CNN
+F 0 "#PWR09" H 7900 1050 50  0001 C CNN
 F 1 "+3.3V" H 7900 1340 50  0000 C CNN
 F 2 "" H 7900 1200 50  0000 C CNN
@@
 $EndComp
 $Comp
-L GND #PWR28
+L GND #PWR010
 U 1 1 574EBFC1
 P 8550 2400
-F 0 "#PWR28" H 8550 2150 50  0001 C CNN
+F 0 "#PWR010" H 8550 2150 50  0001 C CNN
 F 1 "GND" H 8550 2250 50  0000 C CNN
 F 2 "" H 8550 2400 50  0000 C CNN
@@
 $EndComp
 $Comp
-L +3.3V #PWR27
+L +3.3V #PWR011
 U 1 1 574EC177
 P 8550 2100
-F 0 "#PWR27" H 8550 1950 50  0001 C CNN
+F 0 "#PWR011" H 8550 1950 50  0001 C CNN
 F 1 "+3.3V" H 8550 2240 50  0000 C CNN
 F 2 "" H 8550 2100 50  0000 C CNN
@@
 $EndComp
 $Comp
-L +3.3V #PWR8
+L +3.3V #PWR012
 U 1 1 5752AF07
 P 6050 750
-F 0 "#PWR8" H 6050 600 50  0001 C CNN
+F 0 "#PWR012" H 6050 600 50  0001 C CNN
 F 1 "+3.3V" H 6050 890 50  0000 C CNN
 F 2 "" H 6050 750 50  0000 C CNN
@@
 $EndComp
 $Comp
-L GND #PWR15
+L GND #PWR013
 U 1 1 58E603FD
 P 7350 2800
-F 0 "#PWR15" H 7350 2550 50  0001 C CNN
+F 0 "#PWR013" H 7350 2550 50  0001 C CNN
 F 1 "GND" H 7350 2650 50  0000 C CNN
 F 2 "" H 7350 2800 50  0000 C CNN
@@
 $EndComp
 $Comp
-L GND #PWR17
+L GND #PWR014
 U 1 1 58E60435
 P 7350 3200
-F 0 "#PWR17" H 7350 2950 50  0001 C CNN
+F 0 "#PWR014" H 7350 2950 50  0001 C CNN
 F 1 "GND" H 7350 3050 50  0000 C CNN
 F 2 "" H 7350 3200 50  0000 C CNN
@@
 $EndComp
 $Comp
-L +3.3V #PWR14
+L +3.3V #PWR015
 U 1 1 58E6046D
 P 7350 2700
-F 0 "#PWR14" H 7350 2550 50  0001 C CNN
+F 0 "#PWR015" H 7350 2550 50  0001 C CNN
 F 1 "+3.3V" H 7350 2840 50  0000 C CNN
 F 2 "" H 7350 2700 50  0000 C CNN
@@
 $EndComp
 $Comp
-L +3.3V #PWR16
+L +3.3V #PWR016
 U 1 1 58E604A5
 P 7350 3100
-F 0 "#PWR16" H 7350 2950 50  0001 C CNN
+F 0 "#PWR016" H 7350 2950 50  0001 C CNN
 F 1 "+3.3V" H 7350 3240 50  0000 C CNN
 F 2 "" H 7350 3100 50  0000 C CNN
@@
 $EndComp
 $Comp
-L +3.3V #PWR13
+L +3.3V #PWR017
 U 1 1 58E60906
 P 6800 3750
-F 0 "#PWR13" H 6800 3600 50  0001 C CNN
+F 0 "#PWR017" H 6800 3600 50  0001 C CNN
 F 1 "+3.3V" H 6800 3890 50  0000 C CNN
 F 2 "" H 6800 3750 50  0000 C CNN
@@
 $EndComp
 $Comp
-L GND #PWR12
+L GND #PWR018
 U 1 1 58E6093E
 P 6800 3550
-F 0 "#PWR12" H 6800 3300 50  0001 C CNN
+F 0 "#PWR018" H 6800 3300 50  0001 C CNN
 F 1 "GND" H 6800 3400 50  0000 C CNN
 F 2 "" H 6800 3550 50  0000 C CNN
@@
 NoConn ~ 5350 3000
 $Comp
-L GND #PWR10
+L GND #PWR019
 U 1 1 58E616E4
 P 6450 2300
-F 0 "#PWR10" H 6450 2050 50  0001 C CNN
+F 0 "#PWR019" H 6450 2050 50  0001 C CNN
 F 1 "GND" H 6450 2150 50  0000 C CNN
 F 2 "" H 6450 2300 50  0000 C CNN
@@
 $EndComp
 $Comp
-L +3.3V #PWR11
+L +3.3V #PWR020
 U 1 1 58E618C6
 P 6450 3300
-F 0 "#PWR11" H 6450 3150 50  0001 C CNN
+F 0 "#PWR020" H 6450 3150 50  0001 C CNN
 F 1 "+3.3V" H 6450 3440 50  0000 C CNN
 F 2 "" H 6450 3300 50  0000 C CNN
@@
 $EndComp
 $Comp
-L GND #PWR9
+L GND #PWR021
 U 1 1 58E62F9A
 P 6050 4550
-F 0 "#PWR9" H 6050 4300 50  0001 C CNN
+F 0 "#PWR021" H 6050 4300 50  0001 C CNN
 F 1 "GND" H 6050 4400 50  0000 C CNN
 F 2 "" H 6050 4550 50  0000 C CNN
@@
 $EndComp
 $Comp
-L GND #PWR20
+L GND #PWR022
 U 1 1 58E668C3
 P 8100 3450
-F 0 "#PWR20" H 8100 3200 50  0001 C CNN
+F 0 "#PWR022" H 8100 3200 50  0001 C CNN
 F 1 "GND" H 8100 3300 50  0000 C CNN
 F 2 "" H 8100 3450 50  0000 C CNN
@@
 $EndComp
 $Comp
-L GND #PWR21
+L GND #PWR023
 U 1 1 58E6696D
 P 8200 3450
-F 0 "#PWR21" H 8200 3200 50  0001 C CNN
+F 0 "#PWR023" H 8200 3200 50  0001 C CNN
 F 1 "GND" H 8200 3300 50  0000 C CNN
 F 2 "" H 8200 3450 50  0000 C CNN
@@
 $EndComp
 $Comp
-L GND #PWR22
+L GND #PWR024
 U 1 1 58E669C8
 P 8300 3450
-F 0 "#PWR22" H 8300 3200 50  0001 C CNN
+F 0 "#PWR024" H 8300 3200 50  0001 C CNN
 F 1 "GND" H 8300 3300 50  0000 C CNN
 F 2 "" H 8300 3450 50  0000 C CNN
@@
 $EndComp
 $Comp
-L +5V #PWR24
+L +5V #PWR025
 U 1 1 58E66A11
 P 8400 3950
-F 0 "#PWR24" H 8400 3800 50  0001 C CNN
+F 0 "#PWR025" H 8400 3800 50  0001 C CNN
 F 1 "+5V" H 8400 4090 50  0000 C CNN
 F 2 "" H 8400 3950 50  0000 C CNN
@@
 $EndComp
 $Comp
-L +5V #PWR26
+L +5V #PWR026
 U 1 1 58E66A5F
 P 8500 3950
-F 0 "#PWR26" H 8500 3800 50  0001 C CNN
+F 0 "#PWR026" H 8500 3800 50  0001 C CNN
 F 1 "+5V" H 8500 4090 50  0000 C CNN
 F 2 "" H 8500 3950 50  0000 C CNN
@@
 $EndComp
 $Comp
-L +5V #PWR25
+L +5V #PWR027
 U 1 1 58E66ABA
 P 8500 3450
-F 0 "#PWR25" H 8500 3300 50  0001 C CNN
+F 0 "#PWR027" H 8500 3300 50  0001 C CNN
 F 1 "+5V" H 8500 3590 50  0000 C CNN
 F 2 "" H 8500 3450 50  0000 C CNN
@@
 $EndComp
 $Comp
-L +3.3V #PWR23
+L +3.3V #PWR028
 U 1 1 58E66B03
 P 8400 3450
-F 0 "#PWR23" H 8400 3300 50  0001 C CNN
+F 0 "#PWR028" H 8400 3300 50  0001 C CNN
 F 1 "+3.3V" H 8400 3590 50  0000 C CNN
 F 2 "" H 8400 3450 50  0000 C CNN
@@
 	2200 2700 2200 3500
 Connection ~ 2650 3600
-Wire Wire Line
-	3450 2150 3450 2250
-Connection ~ 3450 2150
-Connection ~ 3450 1800
-Wire Wire Line
-	3450 1800 3450 1900
 Wire Wire Line
 	5350 1800 7000 1800
@@
 Wire Wire Line
 	7900 1800 7900 1200
+NoConn ~ 3450 1900
+NoConn ~ 3450 2250
 $EndSCHEMATC

Commit message: Update routing again
Signed-off-by: Leon Anavi <leon@anavi.org>
Connections:
- net +3V3: now also RASP_CONN1.17 (VDD(3.3V))
- net at RASP_CONN1.11 (GPIO17): now also P4.5 (P5); no longer P4.3 (P3)
- net at RASP_CONN1.13 (GPIO27): now also P4.3 (P3); no longer P4.5 (P5)
- no-connect marks 15 -> 14
Changed lines of the file:
@@
 	8100 4150 8100 3950
-Wire Wire Line
-	5350 4050 8200 4050
-Wire Wire Line
-	8200 4050 8200 3950
-Wire Wire Line
-	5350 5050 8300 5050
-Wire Wire Line
-	8300 5050 8300 3950
 Wire Wire Line
 	6100 3450 6100 3650
@@
 	7900 1800 7900 1200
 NoConn ~ 3450 1900
-NoConn ~ 3450 2250
+Connection ~ 3450 2150
+Wire Wire Line
+	3450 2150 3450 2250
+Wire Wire Line
+	5350 5050 8200 5050
+Wire Wire Line
+	8200 5050 8200 3950
+Wire Wire Line
+	5350 4050 8300 4050
+Wire Wire Line
+	8300 4050 8300 3950
 $EndSCHEMATC

Commit message: Add junction between 5V pins on the header
Signed-off-by: Leon Anavi <leon@anavi.org>
Connections:
- net +5V: now also RASP_CONN1.4 (Vpp(5V))
- no-connect marks 14 -> 13
Changed lines of the file:
@@
 Wire Wire Line
 	7900 1800 7900 1200
-NoConn ~ 3450 1900
 Connection ~ 3450 2150
 Wire Wire Line
@@
 Wire Wire Line
 	8300 4050 8300 3950
+Connection ~ 3450 1800
+Wire Wire Line
+	3450 1900 3450 1800
 $EndSCHEMATC

Commit message: Revision 1.1
Revision 1.1 contains these improvements:
* Fixed 1-wire connection for DS18B20 sensor
* Swap GND and 3.3V for analog sensors
* Update text labels

Signed-off-by: Leon Anavi <leon@anavi.org>
Connections:
- net +3V3: now also P2.3 (P3), P3.3 (P3), R5.1; no longer P2.2 (P2), P3.2 (P2)
- net GND: now also P2.2 (P2), P3.2 (P2); no longer P2.3 (P3), P3.3 (P3)
- net at R5.2, RASP_CONN1.7 (GPIO4/GPCLK0): now also P1.2 (P2)
Other:
- moved on the sheet: R5
Changed lines of the file:
@@
 $EndComp
 $Comp
-L GND #PWR013
-U 1 1 58E603FD
-P 7350 2800
-F 0 "#PWR013" H 7350 2550 50  0001 C CNN
-F 1 "GND" H 7350 2650 50  0000 C CNN
-F 2 "" H 7350 2800 50  0000 C CNN
-F 3 "" H 7350 2800 50  0000 C CNN
-	1    7350 2800
-	1    0    0    -1
-$EndComp
-$Comp
-L GND #PWR014
-U 1 1 58E60435
-P 7350 3200
-F 0 "#PWR014" H 7350 2950 50  0001 C CNN
-F 1 "GND" H 7350 3050 50  0000 C CNN
-F 2 "" H 7350 3200 50  0000 C CNN
-F 3 "" H 7350 3200 50  0000 C CNN
-	1    7350 3200
-	1    0    0    -1
-$EndComp
-$Comp
-L +3.3V #PWR015
-U 1 1 58E6046D
-P 7350 2700
-F 0 "#PWR015" H 7350 2550 50  0001 C CNN
-F 1 "+3.3V" H 7350 2840 50  0000 C CNN
-F 2 "" H 7350 2700 50  0000 C CNN
-F 3 "" H 7350 2700 50  0000 C CNN
-	1    7350 2700
-	0    -1   -1   0
-$EndComp
-$Comp
-L +3.3V #PWR016
-U 1 1 58E604A5
-P 7350 3100
-F 0 "#PWR016" H 7350 2950 50  0001 C CNN
-F 1 "+3.3V" H 7350 3240 50  0000 C CNN
-F 2 "" H 7350 3100 50  0000 C CNN
-F 3 "" H 7350 3100 50  0000 C CNN
-	1    7350 3100
-	0    -1   -1   0
-$EndComp
-$Comp
-L +3.3V #PWR017
+L +3.3V #PWR013
 U 1 1 58E60906
 P 6800 3750
-F 0 "#PWR017" H 6800 3600 50  0001 C CNN
+F 0 "#PWR013" H 6800 3600 50  0001 C CNN
 F 1 "+3.3V" H 6800 3890 50  0000 C CNN
 F 2 "" H 6800 3750 50  0000 C CNN
@@
 $EndComp
 $Comp
-L GND #PWR018
+L GND #PWR014
 U 1 1 58E6093E
 P 6800 3550
-F 0 "#PWR018" H 6800 3300 50  0001 C CNN
+F 0 "#PWR014" H 6800 3300 50  0001 C CNN
 F 1 "GND" H 6800 3400 50  0000 C CNN
 F 2 "" H 6800 3550 50  0000 C CNN
@@
 L R R5
 U 1 1 58E60AC0
-P 6250 3650
-F 0 "R5" V 6330 3650 50  0000 C CNN
-F 1 "4.7K" V 6250 3650 50  0000 C CNN
-F 2 "Resistors_SMD:R_0603_HandSoldering" V 6180 3650 50  0001 C CNN
-F 3 "" H 6250 3650 50  0000 C CNN
-	1    6250 3650
-	0    1    1    0
+P 5900 3600
+F 0 "R5" V 5980 3600 50  0000 C CNN
+F 1 "4.7K" V 5900 3600 50  0000 C CNN
+F 2 "Resistors_SMD:R_0603_HandSoldering" V 5830 3600 50  0001 C CNN
+F 3 "" H 5900 3600 50  0000 C CNN
+	1    5900 3600
+	-1   0    0    1
 $EndComp
 NoConn ~ 5350 3000
 $Comp
-L GND #PWR019
+L GND #PWR015
 U 1 1 58E616E4
 P 6450 2300
-F 0 "#PWR019" H 6450 2050 50  0001 C CNN
+F 0 "#PWR015" H 6450 2050 50  0001 C CNN
 F 1 "GND" H 6450 2150 50  0000 C CNN
 F 2 "" H 6450 2300 50  0000 C CNN
@@
 $EndComp
 $Comp
-L +3.3V #PWR020
+L +3.3V #PWR016
 U 1 1 58E618C6
 P 6450 3300
-F 0 "#PWR020" H 6450 3150 50  0001 C CNN
+F 0 "#PWR016" H 6450 3150 50  0001 C CNN
 F 1 "+3.3V" H 6450 3440 50  0000 C CNN
 F 2 "" H 6450 3300 50  0000 C CNN
@@
 $EndComp
 $Comp
-L GND #PWR021
+L GND #PWR017
 U 1 1 58E62F9A
 P 6050 4550
-F 0 "#PWR021" H 6050 4300 50  0001 C CNN
+F 0 "#PWR017" H 6050 4300 50  0001 C CNN
 F 1 "GND" H 6050 4400 50  0000 C CNN
 F 2 "" H 6050 4550 50  0000 C CNN
@@
 $EndComp
 $Comp
-L GND #PWR022
+L GND #PWR018
 U 1 1 58E668C3
 P 8100 3450
-F 0 "#PWR022" H 8100 3200 50  0001 C CNN
+F 0 "#PWR018" H 8100 3200 50  0001 C CNN
 F 1 "GND" H 8100 3300 50  0000 C CNN
 F 2 "" H 8100 3450 50  0000 C CNN
@@
 $EndComp
 $Comp
-L GND #PWR023
+L GND #PWR019
 U 1 1 58E6696D
 P 8200 3450
-F 0 "#PWR023" H 8200 3200 50  0001 C CNN
+F 0 "#PWR019" H 8200 3200 50  0001 C CNN
 F 1 "GND" H 8200 3300 50  0000 C CNN
 F 2 "" H 8200 3450 50  0000 C CNN
@@
 $EndComp
 $Comp
-L GND #PWR024
+L GND #PWR020
 U 1 1 58E669C8
 P 8300 3450
-F 0 "#PWR024" H 8300 3200 50  0001 C CNN
+F 0 "#PWR020" H 8300 3200 50  0001 C CNN
 F 1 "GND" H 8300 3300 50  0000 C CNN
 F 2 "" H 8300 3450 50  0000 C CNN
@@
 $EndComp
 $Comp
-L +5V #PWR025
+L +5V #PWR021
 U 1 1 58E66A11
 P 8400 3950
-F 0 "#PWR025" H 8400 3800 50  0001 C CNN
+F 0 "#PWR021" H 8400 3800 50  0001 C CNN
 F 1 "+5V" H 8400 4090 50  0000 C CNN
 F 2 "" H 8400 3950 50  0000 C CNN
@@
 $EndComp
 $Comp
-L +5V #PWR026
+L +5V #PWR022
 U 1 1 58E66A5F
 P 8500 3950
-F 0 "#PWR026" H 8500 3800 50  0001 C CNN
+F 0 "#PWR022" H 8500 3800 50  0001 C CNN
 F 1 "+5V" H 8500 4090 50  0000 C CNN
 F 2 "" H 8500 3950 50  0000 C CNN
@@
 $EndComp
 $Comp
-L +5V #PWR027
+L +5V #PWR023
 U 1 1 58E66ABA
 P 8500 3450
-F 0 "#PWR027" H 8500 3300 50  0001 C CNN
+F 0 "#PWR023" H 8500 3300 50  0001 C CNN
 F 1 "+5V" H 8500 3590 50  0000 C CNN
 F 2 "" H 8500 3450 50  0000 C CNN
@@
 $EndComp
 $Comp
-L +3.3V #PWR028
+L +3.3V #PWR024
 U 1 1 58E66B03
 P 8400 3450
-F 0 "#PWR028" H 8400 3300 50  0001 C CNN
+F 0 "#PWR024" H 8400 3300 50  0001 C CNN
 F 1 "+3.3V" H 8400 3590 50  0000 C CNN
 F 2 "" H 8400 3450 50  0000 C CNN
@@
 	6950 2600 7350 2600
 Wire Wire Line
-	6400 3650 6800 3650
-Wire Wire Line
-	5350 3450 6100 3450
-Wire Wire Line
 	5750 2600 5350 2600
 Wire Wire Line
@@
 Wire Wire Line
 	8100 4150 8100 3950
-Wire Wire Line
-	6100 3450 6100 3650
 Wire Wire Line
 	6650 1800 6650 1200
@@
 Wire Wire Line
 	3450 1900 3450 1800
+$Comp
+L GND #PWR025
+U 1 1 58F9E900
+P 7350 3100
+F 0 "#PWR025" H 7350 2850 50  0001 C CNN
+F 1 "GND" H 7350 2950 50  0000 C CNN
+F 2 "" H 7350 3100 50  0000 C CNN
+F 3 "" H 7350 3100 50  0000 C CNN
+	1    7350 3100
+	0    1    1    0
+$EndComp
+$Comp
+L GND #PWR026
+U 1 1 58F9E966
+P 7350 2700
+F 0 "#PWR026" H 7350 2450 50  0001 C CNN
+F 1 "GND" H 7350 2550 50  0000 C CNN
+F 2 "" H 7350 2700 50  0000 C CNN
+F 3 "" H 7350 2700 50  0000 C CNN
+	1    7350 2700
+	0    1    1    0
+$EndComp
+$Comp
+L +3.3V #PWR027
+U 1 1 58F9E9A0
+P 7350 2800
+F 0 "#PWR027" H 7350 2650 50  0001 C CNN
+F 1 "+3.3V" H 7350 2940 50  0000 C CNN
+F 2 "" H 7350 2800 50  0000 C CNN
+F 3 "" H 7350 2800 50  0000 C CNN
+	1    7350 2800
+	-1   0    0    1
+$EndComp
+$Comp
+L +3.3V #PWR028
+U 1 1 58F9E9DA
+P 7350 3200
+F 0 "#PWR028" H 7350 3050 50  0001 C CNN
+F 1 "+3.3V" H 7350 3340 50  0000 C CNN
+F 2 "" H 7350 3200 50  0000 C CNN
+F 3 "" H 7350 3200 50  0000 C CNN
+	1    7350 3200
+	-1   0    0    1
+$EndComp
+$Comp
+L +3.3V #PWR029
+U 1 1 58F9EC4B
+P 5900 3750
+F 0 "#PWR029" H 5900 3600 50  0001 C CNN
+F 1 "+3.3V" H 5900 3890 50  0000 C CNN
+F 2 "" H 5900 3750 50  0000 C CNN
+F 3 "" H 5900 3750 50  0000 C CNN
+	1    5900 3750
+	-1   0    0    1
+$EndComp
+Wire Wire Line
+	5350 3450 6200 3450
+Wire Wire Line
+	6200 3450 6200 3650
+Wire Wire Line
+	6200 3650 6800 3650
+Connection ~ 5900 3450
 $EndSCHEMATC

Commit message: Control 3.3V to sensors through GPIO
Connect the 3.3V of the soil moisture sensors
to GPIO5 and GPIO6 of Raspberry Pi. This way
the sensors will be enabled only during
measurement and their life will be significantly
increased.

Signed-off-by: Leon Anavi <leon@anavi.org>
Connections:
- net +3V3: no longer P2.3 (P3), P3.3 (P3)
- net GPIO5: now reaches RASP_CONN1.29 (GPIO5/GPCLK1)
- net GPIO5: now also P3.3 (P3)
- net GPIO6: now reaches RASP_CONN1.31 (GPIO6/GPCLK2)
- net GPIO6: now also P2.3 (P3)
- no-connect marks 13 -> 11
Changed lines of the file:
@@
 NoConn ~ 5350 4350
 NoConn ~ 5350 4250
-NoConn ~ 5350 3550
-NoConn ~ 5350 3650
 NoConn ~ 5350 3750
 NoConn ~ 5350 3850
@@
 	1    0    0    -1
 $EndComp
+$Comp
+L GND #PWR025
+U 1 1 58F9E900
+P 7350 3100
+F 0 "#PWR025" H 7350 2850 50  0001 C CNN
+F 1 "GND" V 7300 2950 50  0000 C CNN
+F 2 "" H 7350 3100 50  0000 C CNN
+F 3 "" H 7350 3100 50  0000 C CNN
+	1    7350 3100
+	0    1    1    0
+$EndComp
+$Comp
+L GND #PWR026
+U 1 1 58F9E966
+P 7350 2700
+F 0 "#PWR026" H 7350 2450 50  0001 C CNN
+F 1 "GND" V 7300 2550 50  0000 C CNN
+F 2 "" H 7350 2700 50  0000 C CNN
+F 3 "" H 7350 2700 50  0000 C CNN
+	1    7350 2700
+	0    1    1    0
+$EndComp
+$Comp
+L +3.3V #PWR027
+U 1 1 58F9EC4B
+P 5900 3750
+F 0 "#PWR027" H 5900 3600 50  0001 C CNN
+F 1 "+3.3V" H 5900 3890 50  0000 C CNN
+F 2 "" H 5900 3750 50  0000 C CNN
+F 3 "" H 5900 3750 50  0000 C CNN
+	1    5900 3750
+	-1   0    0    1
+$EndComp
+Text Label 5500 3550 0    39   ~ 0
+GPIO5
+Text Label 5500 3650 0    39   ~ 0
+GPIO6
 Wire Wire Line
 	950  3500 800  3500
@@
 Wire Wire Line
 	3450 1900 3450 1800
-$Comp
-L GND #PWR025
-U 1 1 58F9E900
-P 7350 3100
-F 0 "#PWR025" H 7350 2850 50  0001 C CNN
-F 1 "GND" H 7350 2950 50  0000 C CNN
-F 2 "" H 7350 3100 50  0000 C CNN
-F 3 "" H 7350 3100 50  0000 C CNN
-	1    7350 3100
-	0    1    1    0
-$EndComp
-$Comp
-L GND #PWR026
-U 1 1 58F9E966
-P 7350 2700
-F 0 "#PWR026" H 7350 2450 50  0001 C CNN
-F 1 "GND" H 7350 2550 50  0000 C CNN
-F 2 "" H 7350 2700 50  0000 C CNN
-F 3 "" H 7350 2700 50  0000 C CNN
-	1    7350 2700
-	0    1    1    0
-$EndComp
-$Comp
-L +3.3V #PWR027
-U 1 1 58F9E9A0
-P 7350 2800
-F 0 "#PWR027" H 7350 2650 50  0001 C CNN
-F 1 "+3.3V" H 7350 2940 50  0000 C CNN
-F 2 "" H 7350 2800 50  0000 C CNN
-F 3 "" H 7350 2800 50  0000 C CNN
-	1    7350 2800
-	-1   0    0    1
-$EndComp
-$Comp
-L +3.3V #PWR028
-U 1 1 58F9E9DA
-P 7350 3200
-F 0 "#PWR028" H 7350 3050 50  0001 C CNN
-F 1 "+3.3V" H 7350 3340 50  0000 C CNN
-F 2 "" H 7350 3200 50  0000 C CNN
-F 3 "" H 7350 3200 50  0000 C CNN
-	1    7350 3200
-	-1   0    0    1
-$EndComp
-$Comp
-L +3.3V #PWR029
-U 1 1 58F9EC4B
-P 5900 3750
-F 0 "#PWR029" H 5900 3600 50  0001 C CNN
-F 1 "+3.3V" H 5900 3890 50  0000 C CNN
-F 2 "" H 5900 3750 50  0000 C CNN
-F 3 "" H 5900 3750 50  0000 C CNN
-	1    5900 3750
-	-1   0    0    1
-$EndComp
 Wire Wire Line
 	5350 3450 6200 3450
@@
 	6200 3650 6800 3650
 Connection ~ 5900 3450
+Wire Wire Line
+	5500 3550 5350 3550
+Wire Wire Line
+	5500 3650 5350 3650
+Text Label 7050 3200 0    39   ~ 0
+GPIO5
+Wire Wire Line
+	7350 3200 7050 3200
+Text Label 7050 2800 0    39   ~ 0
+GPIO6
+Wire Wire Line
+	7350 2800 7050 2800
 $EndSCHEMATC

Commit message: Gardening-pHAT.*: Remap symbols
Remap symbols for newer KiCad version.

Signed-off-by: Leon Anavi <leon@anavi.org>
Parts:
- C1: symbol C -> Gardening-pHAT-rescue:C
- D1: symbol LED -> Gardening-pHAT-rescue:LED
- JP1: symbol JUMPER -> Gardening-pHAT-rescue:JUMPER
- P1, P2, P3: symbol CONN_01X03 -> Gardening-pHAT-rescue:CONN_01X03
- P4: symbol CONN_02X05 -> Gardening-pHAT-rescue:CONN_02X05
- R1, R2, R3, R4, R5, R6, R7: symbol R -> Gardening-pHAT-rescue:R
- RASP_CONN1: symbol Raspberry_PI -> Gardening-pHAT-rescue:Raspberry_PI
- SENS1, SENS2: symbol I2C_SENS_1 -> Gardening-pHAT-rescue:I2C_SENS_1
- U1: symbol CAT24C32WI-GT3 -> Gardening-pHAT-rescue:CAT24C32WI-GT3
- U2: symbol MCP3002 -> Gardening-pHAT-rescue:MCP3002
- UART1: symbol CONN_01X04 -> Gardening-pHAT-rescue:CONN_01X04
